File: hackmit_2025.kicad_pcb (KiCad board)
At the start: 2 copper layers, 2 parts, among them U1 NA555P

Commit message: made some QoL changes
Parts:
- moved U1 38.8 mm to (70.3, 48.8)
- moved D1 37.6 mm to (82.8, 42.8)
Routing:
- net Net-(D1-A): track 66.3 -> 6.36 mm
- net Net-(D1-K): track 30.2 -> 0.00 mm

Commit message: basic functions work, can polish from here
Parts:
- moved D1 12.4 mm to (73.6, 34.5)
- moved U1 7.58 mm to (71.4, 41.3)
Routing:
- net Net-(D1-A): track 6.36 -> 0.00 mm
